File: VHF-FM-2m-TxRx-STM32.kicad_sch (KiCad schematic)
At the start: 0 parts

Commit message: WIP IF PLL charge pump with sufficiently low bandwidth to avoid suppression of injected audio signal.
Parts:
- added C1, C2: C, symbol Device:C
- added Q3, Q4: BFR92P, PCM_Package_TO_SOT_SMD_AKL:SOT-23, symbol PCM_Transistor_BJT_AKL:BFR92P
- added R1: R_US, symbol Device:R_US
- added U1, U2: ADF4002BRUZ, PCM_Package_SO_AKL:TSSOP-16_4.4x5mm_P0.65mm, symbol Timer_PLL:ADF4002BRUZ
- added U3: STM32F103C8Tx, Package_QFP:LQFP-48_7x7mm_P0.5mm, symbol MCU_ST_STM32F1:STM32F103C8Tx
Connections:
- new net: U3.23 (VSS), U3.35 (VSS), U3.47 (VSS)
- new net: C1.2, R1.1
Other:
- note added: "LO PLL and VCO (170 - 174 MHz)"
